File: Hardware/REV-B/ESP32-POE-Wiegand-Relay-REV-B.kicad_sch (KiCad schematic)
At the start: 125 parts, among them IC2 VOD207T, IC3 VOD207T, IC4 THVD1420DR, J2 1984963, J3 0826-1X1T-GH-F, J4 USB_C_Receptacle_USB2.0, J5 1985069, J6 1985001, J8 Conn_01x10, K1 G5Q-1-DC12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

Commit message: update BOM
Parts:
- C11, C14, C15, C16, C18, C24, C? (x2), R1: OldStock Yes -> (none)
- C14, D1, D10, D11, D12, D13, D16, D3, D5, D7, D8, D9, J4, L3, R39, R42, U2: NewPart Yes -> (none)
- J2: LCSC/JLC Part Number NA -> C7467028
- J5: LCSC/JLC Part Number NA -> C7470124
- J6: LCSC/JLC Part Number NA -> C7467032
- K1, K2: LCSC/JLC Part Number NA -> C59752
- PS1: Manufacturer_Name Texas Instruments -> (none); Mouser Price/Stock https://www.mouser.co.uk/ProductDetail/Texas-Instruments/TP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 -> (none); NewPart Yes -> (none)

Commit message: Readme update
Parts:
- R42: value 4.7k/R2512 -> 4.7k/R2512 Populate ONLY for Class 1 PoE See Documentation
Changed lines of the file:
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@@
   (symbol (lib_id "Device:R") (at 118.745 231.14 0) (unit 1)
     (in_bom yes) (on_board yes) (dnp no)
-    (property "Reference" "R42" (at 116.205 233.68 90)
+    (property "Reference" "R42" (at 116.84 221.615 0)
       (effects (font (size 1.27 1.27)) (justify left))
     )
-    (property "Value" "4.7k/R2512" (at 122.555 237.49 90)
-      (effects (font (size 1.27 1.27)) (justify left))
+    (property "Value" "4.7k/R2512 Populate ONLY for Class 1 PoE See Documentation" (at 102.235 223.52 0)
+      (effects (font (size 0.8 0.8)) (justify left))
     )
     (property "Footprint" "Resistor_SMD:R_2512_6332Metric" (at 116.967 231.14 90)

Commit message: Update Bornier
Parts:
- J2: footprint SamacSys_Parts:1984963 -> SamacSys_Parts:1985195
- J5: footprint SamacSys_Parts:1985069 -> SamacSys_Parts:1985292
- J6: footprint SamacSys_Parts:1985001 -> SamacSys_Parts:1985234
Changed lines of the file:
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@@
     (stroke (width 0) (type default))
   )
-  (polyline (pts (xy 537.21 403.86) (xy 530.86 403.86))
-    (stroke (width 0) (type default))
-  )
   (wire (pts (xy 455.295 148.59) (xy 455.295 149.86))
     (stroke (width 0) (type default))
@@
     (stroke (width 0) (type default))
   )
-  (polyline (pts (xy 530.86 408.94) (xy 465.455 408.94))
-    (stroke (width 0) (type default))
-  )
   (wire (pts (xy 71.12 175.26) (xy 71.12 176.53))
     (stroke (width 0) (type default))
@@
     (stroke (width 0) (type default))
   )
-  (polyline (pts (xy 530.86 403.86) (xy 465.455 403.86))
-    (stroke (width 0) (type default))
-  )
   (polyline (pts (xy 522.732 358.14) (xy 522.732 353.06))
     (stroke (width 0) (type default))
@@
     (stroke (width 0) (type default))
   )
-  (polyline (pts (xy 530.86 414.02) (xy 465.455 414.02))
-    (stroke (width 0) (type default))
-  )
   (wire (pts (xy 485.14 266.065) (xy 492.76 266.065))
     (stroke (width 0) (type default))
@@
       (effects (font (size 1.27 1.27)) (justify left))
     )
-    (property "Footprint" "SamacSys_Parts:1984963" (at 434.975 407.975 0)
+    (property "Footprint" "SamacSys_Parts:1985195" (at 434.975 407.975 0)
       (effects (font (size 1.27 1.27)) (justify left top) hide)
     )
@@
       (effects (font (size 1.27 1.27)) (justify left))
     )
-    (property "Footprint" "SamacSys_Parts:1985001" (at 434.975 416.865 0)
+    (property "Footprint" "SamacSys_Parts:1985234" (at 434.975 416.865 0)
       (effects (font (size 1.27 1.27)) (justify left top) hide)
     )
@@
       (effects (font (size 1.27 1.27)) (justify left))
     )
-    (property "Footprint" "SamacSys_Parts:1985069" (at 434.975 437.185 0)
+    (property "Footprint" "SamacSys_Parts:1985292" (at 434.975 437.185 0)
       (effects (font (size 1.27 1.27)) (justify left top) hide)
     )

Commit message: Changer Ethernet Connector, add Switch Wiegand/RS485
Parts:
- removed J3: 0826-1X1T-GH-F, SamacSys_Parts:08261X1TGHF, symbol SamacSys_Parts:0826-1X1T-GH-F
- added C16, C17, C19, C8: 22nf 100v 0603, Capacitor_SMD:C_0603_1608Metric, symbol Device:C_Small
- added J1: RJ45_LED_Shielded, SamacSys_Parts:RJ45-TH_R-RJ45R08P-C000, symbol Connector:RJ45_LED_Shielded
- added R40, R41, R44, R45: 75R 0402, Resistor_SMD:R_0402_1005Metric, symbol Device:R
- added SW1: SW_DPDT_x2, Button_Switch_THT:SW_CuK_JS202011CQN_DPDT_Straight, symbol Switch:SW_DPDT_x2
- added TR1: PT61017PEL, SamacSys_Parts:SMD-16_L12.7-W7.0-P1.27-LS9.5-BL, symbol Transformer:PT61017PEL
Connections:
- net GND: now also C2.2; no longer C2.1
- net RD+: now also TR1.3 (TD-)
- net RD-: now also TR1.1 (TD+)
- net TD+: now also TR1.8 (RD-)
- net TD-: now also TR1.6 (RD+)
- net Wiegand_D0/RS485_A: now also SW1.2 (B); no longer R18.1, R28.2
- net Wiegand_D1/RS485_B: now also SW1.5 (B); no longer R31.2, R32.1
- net at C11.1, C13.1, C15.1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: now also TR1.2 (C_TD), TR1.7 (C_RD)
- net at D14.1: now also C8.1, J1.7, J1.8
- net at D14.2: now also C16.1, J1.4, J1.5
- net at U4.2 (LED2/NINTSEL): now also J1.9
- net at U4.3 (LED1/REGOFF): now also J1.12
- net at D15.2: now also C19.1, TR1.15 (C_TX)
- net at D15.1: now also C17.1, TR1.10 (C_RX)
- net at R24.2: now also J1.11
- net at R24.2: now also J1.10
- new net: C8.2, R45.1
- new net: R31.2, SW1.6 (C)
- new net: C19.2, R44.1
- new net: C17.2, R41.1
- new net: C2.1, J1.13, R40.2, R41.2, R44.2, R45.2
- new net: R28.2, SW1.3 (C)
- new net: C16.2, R40.1
- new net: R32.1, SW1.4 (A)
- new net: R18.1, SW1.1 (A)
- new net RX+: J1.2, TR1.14 (TX-)
- new net RX-: J1.1, TR1.16 (TX+)
- new net TX+: J1.6, TR1.9 (RX-)
- new net TX-: J1.3, TR1.11 (RX+)
- no-connect marks 26 -> 20
Other:
- moved on the sheet: C10, C11, C13, C14, C15, C16, C17, C18, C9, D10, D11, D14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
